File: nekometi/matrix.kicad_sch (KiCad schematic)
At the start: 136 parts, among them SW1 Esc, SW10 9, SW11 0, SW12 -, SW13 =, SW14 Bkscp, SW15 Home, SW16 Tab, SW17 q, SW18 w, SW19 e, SW2 1, SW20 r, SW21 t, SW22 y, SW23 u, SW24 i, SW25 o, SW26 p, SW27 [, SW28 ], SW29 | \, SW3 2, SW30 End, SW31 Capslock, SW32 a, SW33 s, SW34 d, SW35 f, SW36 g, SW37 h, SW38 j, SW39 k, SW4 3, SW40 l, SW41 ;, SW42 ', SW43 Enter, SW44 Pg Up, SW45 L Shift, SW46 z, SW47 x, SW48 c, SW49 v, SW5 4, SW50 b, SW51 n, SW52 m, SW53 <, SW54 >, SW55 ?, SW56 R Shift, SW57 Up, SW58 Pg Down, SW59 L Ctrl, SW6 5, SW60 L Win, SW61 L Alt, SW62 Space 7u, SW63 R Ctrl, SW64 Left, SW65 Down, SW66 Right, SW67 Stepped, SW68 L Bkscp, SW69 R Bkscp, SW7 6, SW8 7, SW9 8

Commit message: add
Other:
- moved on the sheet: SW14A
