File: nekometi/nekometi.kicad_pcb (KiCad board)
At the start: 2 copper layers, 304.3 x 94.8 mm, 156 parts, among them J1 JST, SW1 Esc, SW10 9, SW11 0, SW12 -, SW13 =, SW14 Bkscp, SW15 Home, SW16 Tab, SW17 q, SW18 w, SW19 e, SW2 1, SW20 r, SW21 t, SW22 y, SW23 u, SW24 i, SW25 o, SW26 p, SW27 [, SW28 ], SW29 | \, SW3 2, SW30 End, SW31 Capslock, SW32 a, SW33 s, SW34 d, SW35 f, SW36 g, SW37 h, SW38 j, SW39 k, SW4 3, SW40 l, SW41 ;, SW42 ', SW43 Enter, SW44 Pg Up, SW45 L Shift, SW46 z, SW47 x, SW48 c, SW49 v, SW5 4, SW50 b, SW51 n, SW52 m, SW53 <, SW54 >, SW55 ?, SW56 R Shift, SW57 Up, SW58 Pg Down, SW59 L Ctrl, SW6 5, SW60 L Win, SW61 L Alt, SW62 Space 7u, SW63 R Ctrl, SW64 Left, SW65 Down, SW66 Right, SW67 Stepped, SW68 L Bkscp, SW69 R Bkscp, SW7 6, SW8 7, SW9 8, U1 XC6206PxxxMR-Regulator_Linear, U2 STM32F072C8Tx

Commit message: add
Parts:
- moved D67 2.80 mm to (262.7, 20.6)
- moved D65 1.00 mm to (284.6, 87.0)
- moved D14 0.50 mm to (247.7, 14.2)
- turned D66 to 0 degrees
Routing:
- net Row4: track 310.2 -> 303.8 mm
- net Row2: track 379.2 -> 385.4 mm
- net Col14: track 276.9 -> 273.8 mm, vias 5 -> 4
- net Net-(D67-A): track 12.2 -> 9.22 mm
- net Net-(D66-A): track 8.97 -> 11.3 mm
- net Row0: track 388.4 -> 390.6 mm
- net Col11: track 276.0 -> 274.0 mm
- net Row1: track 409.9 -> 411.5 mm
- net Col13: track 304.5 -> 302.8 mm, vias 6 -> 5
- net Net-(D14-A): track 22.1 -> 21.0 mm
- net Col10: track 215.1 -> 214.0 mm
- net Net-(D65-A): track 6.65 -> 5.67 mm
- net Row3: track 296.6 -> 297.3 mm
- net Col12: track 275.2 -> 275.8 mm
